Commit message: homework1: sim rcm by keyboard & joystick

File: CR_ROS-1.0/dobot_gazebo/urdf/cr5_robot_camera.xacro (robot description, xacro)
@@ -51,5 +51,5 @@
                     <alwaysOn>true</alwaysOn>
                     <updateRate>0.0</updateRate>
-                    <cameraName>/camera</cameraName>
+                    <cameraName>${prefix}</cameraName>
                     <imageTopicName>image_raw</imageTopicName>
                     <cameraInfoTopicName>camera_info</cameraInfoTopicName>

File: CR_ROS-1.0/dobot_gazebo/urdf/cr5_robot_instrument.xacro (robot description, xacro)
@@ -2,4 +2,5 @@
 <robot name="cr5_robot" xmlns:xacro="http://ros.org/wiki/xacro">
 <xacro:include filename="$(find dobot_gazebo)/urdf/cr5_robot_camera.xacro"/>
+<link name="world"/>
  <link name="dummy_link" />
  <link name="base_link">
@@ -32,9 +33,4 @@
     </collision>
   </link>
-  <link  name="world"/>
-<joint name="world_joint" type="fixed">
-    <parent link="world" />
-    <child  link="dummy_link" />
-  </joint>
   <joint name="dummy_joint" type="fixed">
     <parent link="dummy_link" />
@@ -297,4 +293,7 @@
   <xacro:property name="camera_offset_y" value="0" />
   <xacro:property name="camera_offset_z" value="0.343" />
+  <xacro:property name="world_camera_offset_x" value="0.3" />
+  <xacro:property name="world_camera_offset_y" value="0.20" />
+  <xacro:property name="world_camera_offset_z" value="0" />
   <!-- Camera -->
   <joint name="camera_joint" type="fixed">
@@ -304,3 +303,15 @@
   </joint>
   <xacro:usb_camera prefix="camera"/>
+  <!-- Camera -->
+  <joint name="world_camera_joint1" type="fixed">
+    <origin xyz="${world_camera_offset_x} -${world_camera_offset_y} -${world_camera_offset_z}" rpy="0 0.3 0.785" />
+    <parent link="world"/>
+    <child link="world_camera_link"/>
+  </joint>
+  <xacro:usb_camera prefix="world_camera"/>
+  <joint name="world_camera_joint2" type="fixed">
+    <origin xyz="-${world_camera_offset_x} ${world_camera_offset_y} ${world_camera_offset_z}" rpy="0.2152591 -0.2106009 -0.8078383" />
+    <parent link="world_camera_link"/>
+    <child link="dummy_link"/>
+  </joint>
 </robot>
