Commit message: Update cr5_robot_instrument.xacro

File: CR_ROS-1.0/dobot_gazebo/urdf/cr5_robot_instrument.xacro (robot description, xacro)
@@ -3,5 +3,13 @@
 <xacro:include filename="$(find dobot_gazebo)/urdf/cr5_robot_camera.xacro"/>
 <link name="world"/>
+<!-- <joint name="world_joint" type="fixed">
+  <parent link="world" />
+  <child  link="dummy_link" />
+</joint> -->
  <link name="dummy_link" />
+ <joint name="dummy_joint" type="fixed">
+  <parent link="dummy_link" />
+  <child  link="base_link" />
+</joint>
  <link name="base_link">
     <inertial>
@@ -33,8 +41,4 @@
     </collision>
   </link>
-  <joint name="dummy_joint" type="fixed">
-    <parent link="dummy_link" />
-    <child  link="base_link" />
-  </joint>
   <link  name="Link1">
     <inertial>
@@ -305,5 +309,5 @@
   <!-- Camera -->
   <joint name="world_camera_joint1" type="fixed">
-    <origin xyz="${world_camera_offset_x} -${world_camera_offset_y} -${world_camera_offset_z}" rpy="0 0.3 0.785" />
+    <origin xyz="0.3 -0.2 0" rpy="0 0.3 0.785" />
     <parent link="world"/>
     <child link="world_camera_link"/>
@@ -311,5 +315,5 @@
   <xacro:usb_camera prefix="world_camera"/>
   <joint name="world_camera_joint2" type="fixed">
-    <origin xyz="-${world_camera_offset_x} ${world_camera_offset_y} ${world_camera_offset_z}" rpy="0.2152591 -0.2106009 -0.8078383" />
+    <origin xyz="-0.0677 0.3535 -0.0209" rpy="0.2152591 -0.2106009 -0.8078383" />
     <parent link="world_camera_link"/>
     <child link="dummy_link"/>
